File: schema/cpu/cpu/cpu.kicad_sch (KiCad schematic)
At the start: 3 parts, among them IC1 W65C02S6TPG-14, J1 DIN41612_02x32_AC

Commit message: wip
Parts:
- removed RN1: R_Network03, Resistor_THT:R_Array_SIP4, symbol Device:R_Network03
- added C1, C2: 100nF, symbol Device:C
- added J2: ~{RES}, Connector_PinHeader_2.54mm:PinHeader_1x02_P2.54mm_Vertical, symbol Connector_Generic:Conn_01x02
- added J3: EXT CLK, Connector_PinHeader_2.54mm:PinHeader_1x02_P2.54mm_Vertical, symbol Connector_Generic:Conn_01x02
- added J4: Conn_02x06_Odd_Even, symbol Connector_Generic:Conn_02x06_Odd_Even
- added R1, R2: 3k3, Resistor_THT:R_Array_SIP4, symbol Device:R
- added SW1: SW_Push, Button_Switch_THT:SW_PUSH_6mm_H4.3mm, symbol Switch:SW_Push
- added U1: DS1813-5, DS1813-5:TO92127P495H695-3, symbol DS1813-5:DS1813-5
- added U2: 74HC393, Package_SO:SOIC-20W_7.5x12.8mm_P1.27mm, symbol 74xx:74LS393
- added Y1: CXO_DIP8, Oscillator:Oscillator_DIP-8, symbol Oscillator:CXO_DIP8
Connections:
- net +5V: now also C1.2, C2.2, R1.1, R2.1, U1.2 (VCC), U2.14 (VCC), Y1.8 (Vcc); no longer IC1.36 (BE)
- net GND: now also C1.1, C2.1, J2.2 (Pin_2), J3.1 (Pin_1), SW1.1, U1.3 (GND), U2.12 (MR), U2.13 (CP), U2.2 (MR), U2.7 (GND), Y1.4 (GND)
- net PHI2: now also J4.10 (Pin_10), J4.12 (Pin_12), J4.2 (Pin_2), J4.4 (Pin_4), J4.6 (Pin_6), J4.8 (Pin_8)
- net R/W: now also J1.c4 (Pin_c4)
- net ~{IRQ}: now also R1.2
- net ~{NMI}: now also R2.2
- net ~{RES}: now also J2.1 (Pin_1), SW1.2, U1.1 (~{RST})
- net RDY: now reaches IC1.2 (RDY)
- net RDY: now also J1.a2 (Pin_a2)
- net BE: now reaches J1.a25 (Pin_a25)
- net BE: now also IC1.36 (BE)
- new net: J4.1 (Pin_1), U2.1 (CP), Y1.5 (OUT)
- new net: J3.2 (Pin_2), J4.11 (Pin_11)
- new net: J4.3 (Pin_3), U2.3 (Q0)
- new net: J4.5 (Pin_5), U2.4 (Q1)
- new net: J4.7 (Pin_7), U2.5 (Q2)
- new net: J4.9 (Pin_9), U2.6 (Q3)
- no-connect marks 4 -> 37
Other:
- note added: "A déporter sur la backplate"
- note added: "CPU"
- note added: "Clock"
- note added: "Reset"
- moved on the sheet: IC1, J1

Commit message: wip
Parts:
- added C3, C4: 100nF, symbol Device:C
Connections:
- net +5V: now also C3.2, C4.2
- net GND: now also C3.1, C4.1
- no-connect marks 37 -> 38
Other:
- note added: "BUS"

Commit message: wip
Parts:
- C1, C2, C3, C4: footprint (none) -> Capacitor_THT:C_Rect_L4.0mm_W2.5mm_P2.50mm
Changed lines of the file:
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@@
 			)
 		)
-		(property "Footprint" ""
+		(property "Footprint" "Capacitor_THT:C_Rect_L4.0mm_W2.5mm_P2.50mm"
 			(at 248.92 54.9148 0)
 			(hide yes)
@@
 			)
 		)
-		(property "Footprint" ""
+		(property "Footprint" "Capacitor_THT:C_Rect_L4.0mm_W2.5mm_P2.50mm"
 			(at 100.33 90.4748 0)
 			(hide yes)
@@
 			)
 		)
-		(property "Footprint" ""
+		(property "Footprint" "Capacitor_THT:C_Rect_L4.0mm_W2.5mm_P2.50mm"
 			(at 100.33 84.1248 0)
 			(hide yes)
@@
 			)
 		)
-		(property "Footprint" ""
+		(property "Footprint" "Capacitor_THT:C_Rect_L4.0mm_W2.5mm_P2.50mm"
 			(at 236.22 151.4348 0)
 			(hide yes)
