File: schema/backplate/backplate/backplate.kicad_sch (KiCad schematic)
At the start: 8 parts, among them J1 DIN41612_02x32_AC, J2 DIN41612_02x32_AC, J3 DIN41612_02x32_AC, J4 DIN41612_02x32_AC, J5 DIN41612_02x32_AC, J6 DIN41612_02x32_AC, J7 DIN41612_02x32_AC, J8 DIN41612_02x32_AC

Commit message: wip
Parts:
- added C1, C2, C3, C4, C5, C6, C7, C8: 100nF, Capacitor_THT:C_Rect_L4.0mm_W2.5mm_P2.50mm, symbol Device:C_Small
- added C10, C11, C12, C13, C14, C15, C16, C9: 10uF, Package_LCC:PLCC-44_16.6x16.6mm_P1.27mm, symbol Device:C_Polarized_Small
- added J9: ~{RES}, Connector_PinHeader_2.54mm:PinHeader_1x02_P2.54mm_Vertical, symbol Connector_Generic:Conn_01x02
- added R1, R2, R3: 3k3, symbol Device:R
- added SW1: SW_Push, Button_Switch_THT:SW_PUSH_6mm_H4.3mm, symbol Switch:SW_Push
Connections:
- net +5V: now also C1.1, C10.1, C11.1, C12.1, C13.1, C14.1, C15.1, C16.1, C2.1, C3.1, C4.1, C5.1, C6.1, C7.1, C8.1, C9.1, R1.1, R2.1, R3.1
- net BE: now also R2.2
- net GND: now also C1.2, C10.2, C11.2, C12.2, C13.2, C14.2, C15.2, C16.2, C2.2, C3.2, C4.2, C5.2, C6.2, C7.2, C8.2, C9.2, J9.2 (Pin_2), SW1.1
- net RDY: now also R3.2
- net ~{RES}: now also J9.1 (Pin_1), R1.2, SW1.2
Other:
- note added: "PULLUPS"
- note added: "RESET"

Commit message: wip
Parts:
- added C17: 1000uF, Capacitor_THT:CP_Radial_D10.0mm_P5.00mm, symbol Device:C_Polarized
- added F1: Polyfuse, Fuse:Fuse_Littelfuse-LVR100, symbol Device:Polyfuse
- added J10: POWER, symbol Connector_Generic:Conn_01x02
- added J11: PWR_BUTTON, symbol Connector_Generic:Conn_01x02
- added Q1: IRF9540N, Package_TO_SOT_THT:TO-220-3_Vertical, symbol Transistor_FET:IRF9540N
- added SW2: PWR_BUTTON, Button_Switch_THT:SW_Push_2P2T_Toggle_CK_PVA2xxH2xxxxxxV2, symbol Switch:SW_SPST
Connections:
- net +5V: now also C17.1, J11.2 (Pin_2), SW2.2 (B)
- net GND: now also C17.2, J10.1 (Pin_1), Q1.1 (G)
- new net: F1.1, J10.2 (Pin_2)
- new net: F1.2, Q1.2 (D)
- new net: J11.1 (Pin_1), Q1.3 (S), SW2.1 (A)
Other:
- note added: "DECOUPLING"
- note added: "POWER"
